Commit message: Fix URDF to use bounded revolute joints.

File: kortex_description/arms/gen3/7dof/urdf/GEN3_URDF_V12.urdf (robot description, URDF)
Before this commit: robot GEN3_URDF_V12, 9 links, 8 joints
Joints:
- joint Actuator1: limit effort=39 velocity=0.8727 -> lower=-6.28318530718 upper=6.28318530718 effort=39 velocity=0.8727; type continuous -> revolute
- joint Actuator3: limit effort=39 velocity=0.8727 -> lower=-6.28318530718 upper=6.28318530718 effort=39 velocity=0.8727; type continuous -> revolute
- joint Actuator5: limit effort=9 velocity=0.8727 -> lower=-6.28318530718 upper=6.28318530718 effort=9 velocity=0.8727; type continuous -> revolute
- joint Actuator7: limit effort=9 velocity=0.8727 -> lower=-6.28318530718 upper=6.28318530718 effort=9 velocity=0.8727; type continuous -> revolute
